File: fanboard3.kicad_pcb (KiCad board)
At the start: 2 copper layers, 65 x 56 mm, 34 parts, among them J1 PWR IN, J11 USB_A, J12 Conn_01x02_Male, J2 Conn_02x08_Odd_Even, J3 Conn_01x10_Male, J6 FAN1, J7 FAN2, J8 FAN3, J9 FAN4, K1 G6K-2, M1 5V, M2 12V, P1 Conn_02x20_Odd_Even, Q1 2SD1047, U1 SN74HCT245, U2 MCP3008

Commit message: Updates
Parts:
- removed D2: D, Diodes_SMD:D_SMA
- removed Q1: 2SD1047, TO_SOT_Packages_SMD:SOT-223
- removed R10, R12, R8: 10K, Resistors_SMD:R_1210_HandSoldering
- removed R11, R7, R9: 100K, Resistors_SMD:R_1210_HandSoldering
- removed U2: MCP3008, Housings_SSOP:SOP-16_4.4x10.4mm_Pitch1.27mm
- R5: value 1K -> 150
- R6: value 1K -> 0
- moved R4 31.9 mm to (250.7, 113.8), turned to 270 degrees
- moved J12 24.8 mm to (203.3, 136.2)
- moved R5 13.9 mm to (237.8, 122.1), turned to 180 degrees
- moved D1 13.3 mm to (229.0, 131.2)
- moved K1 2.83 mm to (237.6, 130.4), turned to 0 degrees
- moved R6 2.26 mm to (246.1, 113.9)
- moved U1 1.30 mm to (237.4, 113.9)
- moved R3 0.14 mm to (262.0, 105.3)
- moved R1 0.14 mm to (253.0, 105.3)
- moved R2 0.10 mm to (257.5, 105.4)
Connections:
- K1 pad 1: +5V -> Net-(K1-Pad1)
- K1 pad 5: Net-(K1-Pad5) -> Net-(D1-Pad1)
- K1 pad 6: Net-(K1-Pad6) -> GND
- K1 pad 8: Net-(D1-Pad1) -> GND
- P1 pad 11: GPIO17 -> /GPIO17(GEN0)
- P1 pad 35: MISO -> /GPIO19(SPI1_MISO)
- P1 pad 38: MOSI -> /GPIO20(SPI1_MOSI)
- P1 pad 40: SCLK -> /GPIO21(SPI1_SCK)
- R6 pad 1: Net-(Q1-Pad1) -> RELAY
- R6 pad 2: RELAY -> Net-(K1-Pad1)
Routing:
- net +3V3: track 175.2 -> 71.6 mm
- net SCLK: track 67.5 -> 0.00 mm
- net MOSI: track 62.6 -> 0.00 mm
- net MISO: track 57.8 -> 0.00 mm
- net B1: track 65.0 -> 14.8 mm
- net GPIO17: track 49.4 -> 0.00 mm, vias 2 -> 0
- net GND: track 277.3 -> 228.1 mm
- net +5V: track 131.2 -> 91.0 mm, vias 0 -> 1
- net Net-(R11-Pad2): track 38.0 -> 0.00 mm
- net Net-(R10-Pad1): track 31.9 -> 0.00 mm
- net +12V: track 137.0 -> 105.4 mm, vias 1 -> 0
- net Net-(K1-Pad1): track 0.00 -> 27.5 mm
- net NO: track 35.6 -> 59.3 mm
- net Net-(Q1-Pad1): track 21.3 -> 0.00 mm
- net Net-(R7-Pad2): track 19.9 -> 0.00 mm
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Other:
- board text added: "+12V"
- board text added: "PWM"
- board text added: "RPI 3D PRINTER AUX BOARD V1.3"
- board text added: "RPM"
- board text removed: "RPI 3D PRINTER AUX BOARD V1.2"
