File: fanboard3.sch (KiCad schematic (older format))
At the start: 25 parts, among them J1 PWR IN, J11 USB_A, J12 Conn_01x02_Male, J2 Conn_02x08_Odd_Even, J3 Conn_01x10_Male, J6 FAN1, J7 FAN2, J8 FAN3, J9 FAN4, K1 G6K-2, M1 5V, M2 12V, P1 Conn_02x20_Odd_Even, U1 SN74HCT245

Commit message: Updates
Parts:
- M1, M2: symbol ali-stuff:LM2596BuckConverterModule -> fanboard3-rescue:LM2596BuckConverterModule-ali-stuff
Changed lines of the file:
@@
 	1200 4325 1475 4325
 $Comp
-L ali-stuff:LM2596BuckConverterModule M1
+L fanboard3-rescue:LM2596BuckConverterModule-ali-stuff M1
 U 1 1 6031FD7D
 P 2925 4525
@@
 $EndComp
 $Comp
-L ali-stuff:LM2596BuckConverterModule M2
+L fanboard3-rescue:LM2596BuckConverterModule-ali-stuff M2
 U 1 1 6032064A
 P 2925 3625
